Commit message: Add a new launch file and add damping to the joints

File: kinova_description/urdf/kinova_common.xacro (robot description, xacro)
@@ -51,5 +51,5 @@
         <limit effort="2000" velocity="1" lower="${joint_lower_limit}" upper="${joint_upper_limit}"/>
         <origin xyz="${joint_origin_xyz}" rpy="${joint_origin_rpy}"/>
-        <dynamics damping="0.0" friction="0.0"/>
+        <dynamics damping=".2" friction=".0"/>
      </joint>
    <xacro:unless value="${fixed}">
